File: hw/eagle/bc-led_pwm-universal.brd (EAGLE design)
At the start: 100 x 80 mm, 103 parts, among them T1 IRF7413, T10 IRF7413, T11 IRF7413, T12 IRF7413, T13 IRF7413, T14 IRF7413, T15 IRF7413, T16 IRF7413, T2 IRF7413, T3 IRF7413, T4 IRF7413, T5 IRF7413, T6 IRF7413, T7 IRF7413, T8 IRF7413, T9 IRF7413

Commit message: added names and partlist
Parts:
- renumbered U$18 to JP2B, U$28 to JP2C, U$38 to JP2D, U$7 to JP1, U$8 to JP2A
Changed lines of the file:
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@@
 <attribute name="VALUE" x="29.21" y="12.065" size="1.27" layer="28" rot="MR270"/>
 </element>
-<element name="U$7" library="mixi" package="HDR-5.08-1_2" value="STLZ950/2G-5.08-H" x="3.81" y="15.24" smashed="yes" rot="R180"/>
-<element name="U$8" library="mixi" package="HDR-5.08-1_4" value="STLZ950/4G-5.08-V" x="19.05" y="3.81" smashed="yes" rot="R90"/>
+<element name="JP1" library="mixi" package="HDR-5.08-1_2" value="STLZ950/2G-5.08-H" x="3.81" y="15.24" smashed="yes" rot="R180"/>
+<element name="JP2A" library="mixi" package="HDR-5.08-1_4" value="STLZ950/4G-5.08-V" x="19.05" y="3.81" smashed="yes" rot="R90"/>
 <element name="T5" library="mixi" package="SO8" value="IRF7413" x="31.75" y="12.7" smashed="yes" rot="R180">
 <attribute name="NAME" x="31.115" y="12.065" size="1.27" layer="25"/>
@@
 <attribute name="VALUE" x="49.53" y="12.065" size="1.27" layer="28" rot="MR270"/>
 </element>
-<element name="U$18" library="mixi" package="HDR-5.08-1_4" value="STLZ950/4G-5.08-V" x="39.37" y="3.81" smashed="yes" rot="R90"/>
+<element name="JP2B" library="mixi" package="HDR-5.08-1_4" value="STLZ950/4G-5.08-V" x="39.37" y="3.81" smashed="yes" rot="R90"/>
 <element name="T9" library="mixi" package="SO8" value="IRF7413" x="52.07" y="12.7" smashed="yes" rot="R180">
 <attribute name="NAME" x="51.435" y="12.065" size="1.27" layer="25"/>
@@
 <attribute name="VALUE" x="69.85" y="12.065" size="1.27" layer="28" rot="MR270"/>
 </element>
-<element name="U$28" library="mixi" package="HDR-5.08-1_4" value="STLZ950/4G-5.08-V" x="59.69" y="3.81" smashed="yes" rot="R90"/>
+<element name="JP2C" library="mixi" package="HDR-5.08-1_4" value="STLZ950/4G-5.08-V" x="59.69" y="3.81" smashed="yes" rot="R90"/>
 <element name="T13" library="mixi" package="SO8" value="IRF7413" x="72.39" y="12.7" smashed="yes" rot="R180">
 <attribute name="NAME" x="70.485" y="12.065" size="1.27" layer="25"/>
@@
 <attribute name="VALUE" x="90.17" y="12.065" size="1.27" layer="28" rot="MR270"/>
 </element>
-<element name="U$38" library="mixi" package="HDR-5.08-1_4" value="STLZ950/4G-5.08-V" x="80.01" y="3.81" smashed="yes" rot="R90"/>
+<element name="JP2D" library="mixi" package="HDR-5.08-1_4" value="STLZ950/4G-5.08-V" x="80.01" y="3.81" smashed="yes" rot="R90"/>
 <element name="R6" library="resistor" package="R3216" value="0R" x="34.29" y="69.85" smashed="yes" rot="R270">
 <attribute name="NAME" x="33.782" y="67.183" size="1.27" layer="25" rot="R270"/>
@@
 <contactref element="R34" pad="1"/>
 <contactref element="R44" pad="1"/>
-<contactref element="U$7" pad="P$1"/>
+<contactref element="JP1" pad="P$1"/>
 <contactref element="R54" pad="1"/>
 <contactref element="R64" pad="1"/>
@@
 <contactref element="R43" pad="1"/>
 <contactref element="JP3" pad="1"/>
-<contactref element="U$7" pad="P$2"/>
+<contactref element="JP1" pad="P$2"/>
 <wire x1="15.24" y1="14.1" x2="14.04" y2="15.3" width="1.27" layer="1"/>
 <wire x1="14.04" y1="15.3" x2="13.335" y2="15.3" width="1.27" layer="1"/>
@@
 <contactref element="R13" pad="2"/>
 <contactref element="R14" pad="2"/>
-<contactref element="U$8" pad="P$1"/>
+<contactref element="JP2A" pad="P$1"/>
 <wire x1="11.43" y1="3.81" x2="11.43" y2="8.76" width="2.032" layer="16"/>
 <wire x1="9.525" y1="10.1" x2="10.795" y2="10.1" width="1.27" layer="1"/>
@@
 <contactref element="R23" pad="2"/>
 <contactref element="R24" pad="2"/>
-<contactref element="U$8" pad="P$2"/>
+<contactref element="JP2A" pad="P$2"/>
 <wire x1="16.51" y1="3.81" x2="16.51" y2="8.76" width="2.032" layer="16"/>
 <wire x1="20.066" y1="20.19" x2="20.066" y2="20.036" width="1.27" layer="1"/>
@@
 <contactref element="R33" pad="2"/>
 <contactref element="R34" pad="2"/>
-<contactref element="U$8" pad="P$3"/>
+<contactref element="JP2A" pad="P$3"/>
 <wire x1="21.59" y1="3.81" x2="21.59" y2="8.76" width="2.032" layer="16"/>
 <wire x1="19.685" y1="10.1" x2="20.955" y2="10.1" width="1.27" layer="1"/>
@@
 <contactref element="R43" pad="2"/>
 <contactref element="R44" pad="2"/>
-<contactref element="U$8" pad="P$4"/>
+<contactref element="JP2A" pad="P$4"/>
 <wire x1="26.67" y1="3.81" x2="26.67" y2="8.76" width="2.032" layer="16"/>
 <wire x1="24.765" y1="18.99" x2="26.035" y2="18.99" width="1.27" layer="1"/>
@@
 <contactref element="R53" pad="2"/>
 <contactref element="R54" pad="2"/>
-<contactref element="U$18" pad="P$1"/>
+<contactref element="JP2B" pad="P$1"/>
 <wire x1="31.75" y1="3.81" x2="31.75" y2="8.76" width="2.032" layer="16"/>
 <wire x1="29.845" y1="10.1" x2="31.115" y2="10.1" width="1.27" layer="1"/>
@@
 <contactref element="R63" pad="2"/>
 <contactref element="R64" pad="2"/>
-<contactref element="U$18" pad="P$2"/>
+<contactref element="JP2B" pad="P$2"/>
 <wire x1="36.83" y1="3.81" x2="36.83" y2="8.76" width="2.032" layer="16"/>
 <wire x1="34.925" y1="18.99" x2="36.195" y2="18.99" width="1.27" layer="1"/>
@@
 <contactref element="R73" pad="2"/>
 <contactref element="R74" pad="2"/>
-<contactref element="U$18" pad="P$3"/>
+<contactref element="JP2B" pad="P$3"/>
 <wire x1="41.91" y1="3.81" x2="41.91" y2="8.76" width="2.032" layer="16"/>
 <wire x1="40.005" y1="10.1" x2="41.275" y2="10.1" width="1.27" layer="1"/>
@@
 <contactref element="R83" pad="2"/>
 <contactref element="R84" pad="2"/>
-<contactref element="U$18" pad="P$4"/>
+<contactref element="JP2B" pad="P$4"/>
 <wire x1="46.99" y1="3.81" x2="46.99" y2="8.76" width="2.032" layer="16"/>
 <wire x1="45.085" y1="18.99" x2="46.355" y2="18.99" width="1.27" layer="1"/>
@@
 <contactref element="R93" pad="2"/>
 <contactref element="R94" pad="2"/>
-<contactref element="U$28" pad="P$1"/>
+<contactref element="JP2C" pad="P$1"/>
 <wire x1="52.07" y1="3.81" x2="52.07" y2="8.76" width="2.032" layer="16"/>
 <wire x1="50.165" y1="10.1" x2="51.435" y2="10.1" width="1.27" layer="1"/>
@@
 <contactref element="R103" pad="2"/>
 <contactref element="R104" pad="2"/>
-<contactref element="U$28" pad="P$2"/>
+<contactref element="JP2C" pad="P$2"/>
 <wire x1="57.15" y1="3.81" x2="57.15" y2="8.76" width="2.032" layer="16"/>
 <wire x1="55.245" y1="18.99" x2="56.515" y2="18.99" width="1.27" layer="1"/>
@@
 <contactref element="R113" pad="2"/>
 <contactref element="R114" pad="2"/>
-<contactref element="U$28" pad="P$3"/>
+<contactref element="JP2C" pad="P$3"/>
 <wire x1="62.23" y1="3.81" x2="62.23" y2="8.76" width="2.032" layer="16"/>
 <wire x1="60.325" y1="10.1" x2="61.595" y2="10.1" width="1.27" layer="1"/>
@@
 <contactref element="R123" pad="2"/>
 <contactref element="R124" pad="2"/>
-<contactref element="U$28" pad="P$4"/>
+<contactref element="JP2C" pad="P$4"/>
 <wire x1="67.31" y1="3.81" x2="67.31" y2="8.76" width="2.032" layer="16"/>
 <wire x1="70.866" y1="20.19" x2="70.866" y2="20.036" width="1.27" layer="1"/>
@@
 <contactref element="R133" pad="2"/>
 <contactref element="R134" pad="2"/>
-<contactref element="U$38" pad="P$1"/>
+<contactref element="JP2D" pad="P$1"/>
 <wire x1="72.39" y1="3.81" x2="72.39" y2="8.76" width="2.032" layer="16"/>
 <wire x1="70.485" y1="10.1" x2="71.755" y2="10.1" width="1.27" layer="1"/>
@@
 <contactref element="R143" pad="2"/>
 <contactref element="R144" pad="2"/>
-<contactref element="U$38" pad="P$2"/>
+<contactref element="JP2D" pad="P$2"/>
 <wire x1="77.47" y1="3.81" x2="77.47" y2="8.76" width="2.032" layer="16"/>
 <wire x1="75.565" y1="18.99" x2="76.835" y2="18.99" width="1.27" layer="1"/>
@@
 <contactref element="R153" pad="2"/>
 <contactref element="R154" pad="2"/>
-<contactref element="U$38" pad="P$3"/>
+<contactref element="JP2D" pad="P$3"/>
 <wire x1="82.55" y1="3.81" x2="82.55" y2="8.76" width="2.032" layer="16"/>
 <wire x1="80.645" y1="10.1" x2="81.915" y2="10.1" width="1.27" layer="1"/>
@@
 <contactref element="R163" pad="2"/>
 <contactref element="R164" pad="2"/>
-<contactref element="U$38" pad="P$4"/>
+<contactref element="JP2D" pad="P$4"/>
 <wire x1="87.63" y1="3.81" x2="87.63" y2="8.76" width="2.032" layer="16"/>
 <wire x1="85.725" y1="18.99" x2="86.995" y2="18.99" width="1.27" layer="1"/>
