File: hw/eagle/bc-led_pwm-universal.sch (EAGLE design)
At the start: 86 parts, among them T1 IRF7413, T10 IRF7413, T11 IRF7413, T12 IRF7413, T13 IRF7413, T14 IRF7413, T15 IRF7413, T16 IRF7413, T17 FDC6318P, T2 IRF7413, T3 IRF7413, T4 IRF7413, T5 IRF7413, T6 IRF7413, T7 IRF7413, T8 IRF7413, T9 IRF7413

Commit message: rotate core module to have convenient access to USB port, added pull-down resistors on output FETs, proper VDD_OFF handling and added power outage monitoring via P17
Parts:
- removed R2: 560R, resistor:R-EU_R2012
- removed R3: 10k, resistor:R-EU_R2012
- removed T17: FDC6318P, mixi:FDC6318P
- added D2, D3, D4: B340A, diode:DIODE-MELF-MLL41
- added R21, R22, R23, R24, R25, R26, R27, R28, R29, R30, R43, R44, R45, R46, R47, R48: 10k, resistor:R-EU_R3216
- added R49: 560R, resistor:R-EU_R3216
- R1: value 100k -> 560R; device resistor:R-EU_R2012 -> resistor:R-EU_R3216
- R4: device resistor:R-EU_R2012 -> resistor:R-EU_R3216
Connections:
- removed net N$1: R1.2, T17.S1, T17.S2
- removed net N$3: R1.1, R2.2, R3.1, T17.G1, T17.G2
- new net N$14: D2.C, R4.2
- new net N$15: D3.C, R49.2
- net +3V3: now also D2.A, D3.A, D4.A, R1.2; no longer R4.2, T17.D1
- net GND: now also R21.1, R22.1, R23.1, R24.1, R25.1, R26.1, R27.1, R28.1, R29.1, R30.1, R43.1, R44.1, R45.1, R46.1, R47.1, R48.1; no longer R3.2
- net N$10: now also R22.2
- net N$12: now also R24.2
- net N$2: now also R21.2
- net N$22: now also R25.2
- net N$24: now also R26.2
- net N$26: now also R27.2
- net N$28: now also R28.2
- net N$38: now also R29.2
- net N$40: now also R30.2
- net N$42: now also R43.2
- net N$44: now also R44.2
- net N$54: now also R45.2
- net N$56: now also R46.2
- net N$58: now also R47.2
- net N$60: now also R48.2
- net N$8: now also R23.2
- net P16: now also JP3.2
- net P17: now also R1.1; no longer JP3.2
- net VDD: now also D4.C; no longer T17.D2
- net VDD_OFF_IN: now also R49.1; no longer R2.1
Other:
- moved on the sheet: R1, R4

Commit message: added ground plane, reworked step-down
Parts:
- removed R10, R16, R40: 390R, resistor:R-EU_0207/7
- removed R15, R17, R18, R19, R20, R35, R36, R8, R9: 0R, resistor:R-EU_R3216
- removed R26, R28: 10k, resistor:R-EU_R3216
- added R111, R121, R141, R51: 390R, resistor:R-EU_0207/7
- added R112, R122: 10k, resistor:R-EU_R3216
- added R113, R114, R134, R143, R144, R53, R54: 0R, resistor:R-EU_R3216
- added R2: 560R, resistor:R-EU_R3216
- D2, D3, D4: device diode:DIODE-MELF-MLL41 -> diode:PMLL41SOD80C
- L1: device eagle-ltspice:LL3225P -> inductors:BC12
- R11, R41, R81: value 0R -> 390R; device resistor:R-EU_R3216 -> resistor:R-EU_0207/7
- R12, R32, R42, R62: value 0R -> 10k
- R13, R34, R5, R64: value 390R -> 0R; device resistor:R-EU_0207/7 -> resistor:R-EU_R3216
- R21: value 10k -> 390R; device resistor:R-EU_R3216 -> resistor:R-EU_0207/7
- R23, R24, R43, R44: value 10k -> 0R
- R4: value 560R -> 0R
- R82: value 390R -> 10k; device resistor:R-EU_0207/7 -> resistor:R-EU_R3216
- renumbered R25 to R52, R27 to R72, R29 to R92, R30 to R102, R37 to R71, R38 to R73, R39 to R74, R45 to R132, R46 to R142, R47 to R152, R48 to R162, R49 to R3, R55 to R91, R56 to R93, R57 to R94, R58 to R101, R59 to R103, R60 to R104, R65 to R123, R66 to R124, R79 to R131, R80 to R133, R85 to R151, R86 to R153, R87 to R154, R88 to R161, R89 to R163, R90 to R164
Connections:
- net +12V: now also R114.1, R134.1, R14.1, R144.1, R24.1, R34.1, R44.1, R54.1, R64.1; no longer R12.1, R15.1, R18.1, R33.1, R36.1, R42.1, R63.1, R7.1, R81.1
- net BAT_OFF: now also R2.1; no longer R4.1
- net GND: now also R112.1, R113.1, R12.1, R122.1, R13.1, R143.1, R33.1, R42.1, R53.1, R63.1, R82.1; no longer R11.1, R14.1, R17.1, R21.1, R24.1, R26.1, R28.1, R35.1, R41.1, R44.1, R6.1
- net N$10: now also R21.2; no longer R10.2
- net N$11: now also R23.2, R24.2; no longer R11.2, R12.2
- net N$12: now also R41.2, R42.2; no longer R16.2, R24.2
- net N$13: now also R43.2, R44.2; no longer R17.2, R18.2
- net N$14: now also R2.2; no longer R4.2
- net N$2: now also R11.2, R12.2; no longer R21.2, R5.2
- net N$22: now also R51.2; no longer R31.2
- net N$23: now also R53.2, R54.2; no longer R32.2, R33.2
- net N$24: now also R61.2, R62.2; no longer R26.2, R34.2
- net N$25: now also R63.2, R64.2; no longer R35.2, R36.2
- net N$28: now also R81.2, R82.2; no longer R28.2, R40.2
- net N$29: now also R83.2, R84.2; no longer R41.2, R42.2
- net N$4: now also R13.2, R14.2; no longer R6.2, R7.2
- net N$42: now also R111.2, R112.2; no longer R43.2, R61.2
- net N$43: now also R113.2, R114.2; no longer R62.2, R63.2
- net N$44: now also R121.2, R122.2; no longer R44.2, R64.2
- net N$5: now also R5.2, R7.2; no longer R20.2, R9.2
- net N$55: now also R134.2; no longer R81.2
- net N$56: now also R141.2; no longer R82.2
- net N$57: now also R143.2, R144.2; no longer R83.2, R84.2
- net N$6: now also R4.2, R6.2; no longer R19.2, R8.2
- net N$8: now also R31.2, R32.2; no longer R13.2, R23.2
- net N$9: now also R33.2, R34.2; no longer R14.2, R15.2
- net P0: now also R11.1, R4.1; no longer R5.1, R8.1
- net P1: now also R21.1, R5.1; no longer R10.1, R9.1
- net P10: now also R111.1; no longer R61.1
- net P11: now also R121.1; no longer R64.1
- net P13: now also R141.1; no longer R82.1
- net P2: now also R31.1; no longer R13.1
- net P3: now also R41.1; no longer R16.1
- net P4: now also R51.1, R6.1; no longer R19.1, R31.1
- net P5: now also R61.1, R7.1; no longer R20.1, R34.1
- net P7: now also R81.1; no longer R40.1
Other:
- moved on the sheet: C1, R11, R12, R13, R14, R21, R23, R24, R31, R32, R33, R34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

Commit message: Changed 0R on FET gates, fixed symbols for schottky & inductor
Parts:
- D1: device diode:DIODE-MELF-MLL41 -> diode:SCHOTTKY-DIODESMD
- D2, D3, D4: value B340A -> PMLL41SOD80C
- L1: device inductors:BC12 -> mixi-inductors:L-GENERIC-BC12
- R101, R11, R111, R121, R131, R141, R151, R161, R21, R31, R41, R51, R61, R71, R81, R91: value 390R -> 0R
Changed lines of the file:
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@@
 <part name="GND3" library="supply1" deviceset="GND" device=""/>
 <part name="P+2" library="supply1" deviceset="+12V" device=""/>
-<part name="D1" library="diode" deviceset="DIODE-" device="MELF-MLL41" value="B340A"/>
-<part name="L1" library="inductors" deviceset="BC12" device="" value="33uH"/>
+<part name="D1" library="diode" deviceset="SCHOTTKY-DIODE" device="SMD" value="B340A"/>
+<part name="L1" library="mixi-inductors" deviceset="L-GENERIC-BC12" device="" package3d_urn="urn:adsk.eagle:package:15120/1" value="33uH"/>
 <part name="U$1" library="mixi" deviceset="AP1501" device=""/>
 <part name="VDD1" library="supply1" deviceset="VDD" device=""/>
@@
 <part name="R2" library="resistor" deviceset="R-EU_" device="R3216" value="560R"/>
 <part name="T1" library="mixi" deviceset="IRF7413" device=""/>
-<part name="R11" library="resistor" deviceset="R-EU_" device="0207/7" value="390R"/>
+<part name="R11" library="resistor" deviceset="R-EU_" device="0207/7" value="0R"/>
 <part name="GND1" library="supply1" deviceset="GND" device=""/>
 <part name="JP3" library="pinhead" deviceset="PINHD-1X6" device="" value="PCA9685"/>
@@
 <part name="VDD2" library="supply1" deviceset="VDD" device=""/>
 <part name="T2" library="mixi" deviceset="IRF7413" device=""/>
-<part name="R21" library="resistor" deviceset="R-EU_" device="0207/7" value="390R"/>
+<part name="R21" library="resistor" deviceset="R-EU_" device="0207/7" value="0R"/>
 <part name="GND4" library="supply1" deviceset="GND" device=""/>
 <part name="R23" library="resistor" deviceset="R-EU_" device="R3216" value="0R"/>
@@
 <part name="P+3" library="supply1" deviceset="+12V" device=""/>
 <part name="T3" library="mixi" deviceset="IRF7413" device=""/>
-<part name="R31" library="resistor" deviceset="R-EU_" device="0207/7" value="390R"/>
+<part name="R31" library="resistor" deviceset="R-EU_" device="0207/7" value="0R"/>
 <part name="GND5" library="supply1" deviceset="GND" device=""/>
 <part name="R33" library="resistor" deviceset="R-EU_" device="R3216" value="0R"/>
@@
 <part name="P+4" library="supply1" deviceset="+12V" device=""/>
 <part name="T4" library="mixi" deviceset="IRF7413" device=""/>
-<part name="R41" library="resistor" deviceset="R-EU_" device="0207/7" value="390R"/>
+<part name="R41" library="resistor" deviceset="R-EU_" device="0207/7" value="0R"/>
 <part name="GND6" library="supply1" deviceset="GND" device=""/>
 <part name="R43" library="resistor" deviceset="R-EU_" device="R3216" value="0R"/>
@@
 <part name="U$8" library="mixi" deviceset="STLZ950/4G-5.08-V" device=""/>
 <part name="T5" library="mixi" deviceset="IRF7413" device=""/>
-<part name="R51" library="resistor" deviceset="R-EU_" device="0207/7" value="390R"/>
+<part name="R51" library="resistor" deviceset="R-EU_" device="0207/7" value="0R"/>
 <part name="GND12" library="supply1" deviceset="GND" device=""/>
 <part name="R53" library="resistor" deviceset="R-EU_" device="R3216" value="0R"/>
@@
 <part name="P+11" library="supply1" deviceset="+12V" device=""/>
 <part name="T6" library="mixi" deviceset="IRF7413" device=""/>
-<part name="R61" library="resistor" deviceset="R-EU_" device="0207/7" value="390R"/>
+<part name="R61" library="resistor" deviceset="R-EU_" device="0207/7" value="0R"/>
 <part name="GND13" library="supply1" deviceset="GND" device=""/>
 <part name="R63" library="resistor" deviceset="R-EU_" device="R3216" value="0R"/>
@@
 <part name="P+12" library="supply1" deviceset="+12V" device=""/>
 <part name="T7" library="mixi" deviceset="IRF7413" device=""/>
-<part name="R71" library="resistor" deviceset="R-EU_" device="0207/7" value="390R"/>
+<part name="R71" library="resistor" deviceset="R-EU_" device="0207/7" value="0R"/>
 <part name="GND14" library="supply1" deviceset="GND" device=""/>
 <part name="R73" library="resistor" deviceset="R-EU_" device="R3216" value="0R"/>
@@
 <part name="P+13" library="supply1" deviceset="+12V" device=""/>
 <part name="T8" library="mixi" deviceset="IRF7413" device=""/>
-<part name="R81" library="resistor" deviceset="R-EU_" device="0207/7" value="390R"/>
+<part name="R81" library="resistor" deviceset="R-EU_" device="0207/7" value="0R"/>
 <part name="GND15" library="supply1" deviceset="GND" device=""/>
 <part name="R83" library="resistor" deviceset="R-EU_" device="R3216" value="0R"/>
@@
 <part name="U$18" library="mixi" deviceset="STLZ950/4G-5.08-V" device=""/>
 <part name="T9" library="mixi" deviceset="IRF7413" device=""/>
-<part name="R91" library="resistor" deviceset="R-EU_" device="0207/7" value="390R"/>
+<part name="R91" library="resistor" deviceset="R-EU_" device="0207/7" value="0R"/>
 <part name="GND20" library="supply1" deviceset="GND" device=""/>
 <part name="R93" library="resistor" deviceset="R-EU_" device="R3216" value="0R"/>
@@
 <part name="P+19" library="supply1" deviceset="+12V" device=""/>
 <part name="T10" library="mixi" deviceset="IRF7413" device=""/>
-<part name="R101" library="resistor" deviceset="R-EU_" device="0207/7" value="390R"/>
+<part name="R101" library="resistor" deviceset="R-EU_" device="0207/7" value="0R"/>
 <part name="GND21" library="supply1" deviceset="GND" device=""/>
 <part name="R103" library="resistor" deviceset="R-EU_" device="R3216" value="0R"/>
@@
 <part name="P+20" library="supply1" deviceset="+12V" device=""/>
 <part name="T11" library="mixi" deviceset="IRF7413" device=""/>
-<part name="R111" library="resistor" deviceset="R-EU_" device="0207/7" value="390R"/>
+<part name="R111" library="resistor" deviceset="R-EU_" device="0207/7" value="0R"/>
 <part name="GND22" library="supply1" deviceset="GND" device=""/>
 <part name="R113" library="resistor" deviceset="R-EU_" device="R3216" value="0R"/>
@@
 <part name="P+21" library="supply1" deviceset="+12V" device=""/>
 <part name="T12" library="mixi" deviceset="IRF7413" device=""/>
-<part name="R121" library="resistor" deviceset="R-EU_" device="0207/7" value="390R"/>
+<part name="R121" library="resistor" deviceset="R-EU_" device="0207/7" value="0R"/>
 <part name="GND23" library="supply1" deviceset="GND" device=""/>
 <part name="R123" library="resistor" deviceset="R-EU_" device="R3216" value="0R"/>
@@
 <part name="U$28" library="mixi" deviceset="STLZ950/4G-5.08-V" device=""/>
 <part name="T13" library="mixi" deviceset="IRF7413" device=""/>
-<part name="R131" library="resistor" deviceset="R-EU_" device="0207/7" value="390R"/>
+<part name="R131" library="resistor" deviceset="R-EU_" device="0207/7" value="0R"/>
 <part name="GND28" library="supply1" deviceset="GND" device=""/>
 <part name="R133" library="resistor" deviceset="R-EU_" device="R3216" value="0R"/>
@@
 <part name="P+27" library="supply1" deviceset="+12V" device=""/>
 <part name="T14" library="mixi" deviceset="IRF7413" device=""/>
-<part name="R141" library="resistor" deviceset="R-EU_" device="0207/7" value="390R"/>
+<part name="R141" library="resistor" deviceset="R-EU_" device="0207/7" value="0R"/>
 <part name="GND29" library="supply1" deviceset="GND" device=""/>
 <part name="R143" library="resistor" deviceset="R-EU_" device="R3216" value="0R"/>
@@
 <part name="P+28" library="supply1" deviceset="+12V" device=""/>
 <part name="T15" library="mixi" deviceset="IRF7413" device=""/>
-<part name="R151" library="resistor" deviceset="R-EU_" device="0207/7" value="390R"/>
+<part name="R151" library="resistor" deviceset="R-EU_" device="0207/7" value="0R"/>
 <part name="GND30" library="supply1" deviceset="GND" device=""/>
 <part name="R153" library="resistor" deviceset="R-EU_" device="R3216" value="0R"/>
@@
 <part name="P+29" library="supply1" deviceset="+12V" device=""/>
 <part name="T16" library="mixi" deviceset="IRF7413" device=""/>
-<part name="R161" library="resistor" deviceset="R-EU_" device="0207/7" value="390R"/>
+<part name="R161" library="resistor" deviceset="R-EU_" device="0207/7" value="0R"/>
 <part name="GND31" library="supply1" deviceset="GND" device=""/>
 <part name="R163" library="resistor" deviceset="R-EU_" device="R3216" value="0R"/>
@@
 <part name="R162" library="resistor" deviceset="R-EU_" device="R3216" value="10k"/>
 <part name="GND35" library="supply1" deviceset="GND" device=""/>
-<part name="D2" library="diode" deviceset="PMLL41*" device="SOD80C" value="B340A"/>
-<part name="D3" library="diode" deviceset="PMLL41*" device="SOD80C" value="B340A"/>
+<part name="D2" library="diode" deviceset="PMLL41*" device="SOD80C" value=""/>
+<part name="D3" library="diode" deviceset="PMLL41*" device="SOD80C" value=""/>
 <part name="R3" library="resistor" deviceset="R-EU_" device="R3216" value="560R"/>
-<part name="D4" library="diode" deviceset="PMLL41*" device="SOD80C" value="B340A"/>
+<part name="D4" library="diode" deviceset="PMLL41*" device="SOD80C" value=""/>
 <part name="R1" library="resistor" deviceset="R-EU_" device="R3216" value="560R"/>
 </parts>
@@
 </schematic>
 </drawing>
+<compatibility>
+<note version="8.3" severity="warning">
+Since Version 8.3, EAGLE supports URNs for individual library
+assets (packages, symbols, and devices). The URNs of those assets
+will not be understood (or retained) with this version.
+</note>
+<note version="8.3" severity="warning">
+Since Version 8.3, EAGLE supports the association of 3D packages
+with devices in libraries, schematics, and board files. Those 3D
+packages will not be understood (or retained) with this version.
+</note>
+</compatibility>
 </eagle>

Commit message: added names and partlist
Parts:
- renumbered U$18 to JP2B, U$28 to JP2C, U$38 to JP2D, U$7 to JP1, U$8 to JP2A
